File: KiCad/TagBot/regulateur3.3V.kicad_sch (KiCad schematic)
At the start: 5 parts

Commit message: update kicad
Parts:
- gave numbers to parts that had none: 5
Changed lines of the file:
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@@
 		(dnp no)
 		(fields_autoplaced yes)
-		(property "Reference" "U?"
+		(property "Reference" "U501"
 			(at 158.75 93.98 0)
 			(effects
@@
 			(project "TagBot"
 				(path "/6db08f37-7cb3-4000-93f1-ba0d0ffbeb19/f641a0e6-7f59-4351-93f4-c346a0d5b8a7"
-					(reference "U?")
+					(reference "U501")
 					(unit 1)
 				)
@@
 		(dnp no)
 		(fields_autoplaced yes)
-		(property "Reference" "R?"
+		(property "Reference" "R501"
 			(at 200.66 95.885 0)
 			(effects
@@
 			(project "TagBot"
 				(path "/6db08f37-7cb3-4000-93f1-ba0d0ffbeb19/f641a0e6-7f59-4351-93f4-c346a0d5b8a7"
-					(reference "R?")
+					(reference "R501")
 					(unit 1)
 				)
@@
 		(dnp no)
 		(fields_autoplaced yes)
-		(property "Reference" "C?"
+		(property "Reference" "C502"
 			(at 177.8 104.7813 0)
 			(effects
@@
 			(project "TagBot"
 				(path "/6db08f37-7cb3-4000-93f1-ba0d0ffbeb19/f641a0e6-7f59-4351-93f4-c346a0d5b8a7"
-					(reference "C?")
+					(reference "C502")
 					(unit 1)
 				)
@@
 		(dnp no)
 		(fields_autoplaced yes)
-		(property "Reference" "D?"
+		(property "Reference" "D501"
 			(at 201.93 107.6325 90)
 			(effects
@@
 			(project "TagBot"
 				(path "/6db08f37-7cb3-4000-93f1-ba0d0ffbeb19/f641a0e6-7f59-4351-93f4-c346a0d5b8a7"
-					(reference "D?")
+					(reference "D501")
 					(unit 1)
 				)
@@
 		(dnp no)
 		(fields_autoplaced yes)
-		(property "Reference" "C?"
+		(property "Reference" "C501"
 			(at 138.43 103.5113 0)
 			(effects
@@
 			(project "TagBot"
 				(path "/6db08f37-7cb3-4000-93f1-ba0d0ffbeb19/f641a0e6-7f59-4351-93f4-c346a0d5b8a7"
-					(reference "C?")
-					(unit 1)
-				)
+					(reference "C501")
+					(unit 1)
+				)

Commit message: placement pcb
Parts:
- D501: reference (none) -> 150060GS55040
- R501: value 220 -> 100
