File: KiCad/TagBot/regulateur3.3V.kicad_sch (KiCad schematic)
At the start: 5 parts, among them U501 BU33SD5WG-TR

Commit message: placement pcb 2
Changed lines of the file:
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@@
+		(color 0 0 0 0)
+	)
+	(junction
+		(at 175.26 100.33)
+		(diameter 0)
 		(color 0 0 0 0)
 	)
@@
 		(pts
 			(xy 135.89 106.68) (xy 135.89 110.49)
-		)
-		(stroke
-			(width 0)
-			(type default)
-		)
-	)
-	(wire
-		(pts
-			(xy 175.26 100.33) (xy 168.91 100.33)
 		)
 		(stroke
@@
 	(wire
 		(pts
+			(xy 175.26 100.33) (xy 175.26 99.06)
+		)
+		(stroke
+			(width 0)
+			(type default)
+		)
+	)
+	(wire
+		(pts
 			(xy 144.78 102.87) (xy 144.78 100.33)
 		)
@@
 		(pts
 			(xy 175.26 102.87) (xy 175.26 100.33)
+		)
+		(stroke
+			(width 0)
+			(type default)
+		)
+	)
+	(wire
+		(pts
+			(xy 168.91 100.33) (xy 175.26 100.33)
 		)
 		(stroke
@@
 	(hierarchical_label "+3.3V"
 		(shape input)
-		(at 175.26 100.33 90)
+		(at 175.26 99.06 90)
 		(fields_autoplaced yes)
 		(effects

Commit message: update routage
Parts:
- C501, C502: footprint Capacitor_SMD:C_0402_1005Metric -> Capacitor_SMD:C_0603_1608Metric
Changed lines of the file:
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@@
 			)
 		)
-		(property "Footprint" "Capacitor_SMD:C_0402_1005Metric"
+		(property "Footprint" "Capacitor_SMD:C_0603_1608Metric"
 			(at 175.26 105.41 0)
 			(effects
@@
 			)
 		)
-		(property "Footprint" "Capacitor_SMD:C_0402_1005Metric"
+		(property "Footprint" "Capacitor_SMD:C_0603_1608Metric"
 			(at 135.89 104.14 0)
 			(effects
