File: KiCad/TagBot/moteurs.kicad_sch (KiCad schematic)
At the start: 2 parts, among them J1001 Conn_01x06, J1002 Conn_01x06

Commit message: update routage
Connections:
- net LEFT_OUT1: now also J1002.6 (Pin_6); no longer J1002.1 (Pin_1)
- net LEFT_OUT2: now also J1002.1 (Pin_1); no longer J1002.6 (Pin_6)
- net RIGHT_OUT1: now also J1001.6 (Pin_6); no longer J1001.1 (Pin_1)
- net RIGHT_OUT2: now also J1001.1 (Pin_1); no longer J1001.6 (Pin_6)
Changed lines of the file:
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@@
 	(text "Left"
 		(exclude_from_sim no)
-		(at 222.504 148.844 0)
+		(at 225.806 148.59 0)
 		(effects
 			(font
@@
 	(text "Right\n"
 		(exclude_from_sim no)
-		(at 222.504 129.794 0)
+		(at 226.314 129.794 0)
 		(effects
 			(font
@@
 		)
 	)
-	(hierarchical_label "LEFT_OUT2"
+	(hierarchical_label "LEFT_OUT1"
 		(shape input)
 		(at 205.74 156.21 180)
@@
 		)
 	)
-	(hierarchical_label "RIGHT_OUT1"
+	(hierarchical_label "RIGHT_OUT2"
 		(shape input)
 		(at 207.01 124.46 180)
@@
 		)
 	)
-	(hierarchical_label "LEFT_OUT1"
+	(hierarchical_label "LEFT_OUT2"
 		(shape input)
 		(at 205.74 143.51 180)
@@
 		)
 	)
-	(hierarchical_label "RIGHT_OUT2"
+	(hierarchical_label "RIGHT_OUT1"
 		(shape input)
 		(at 207.01 137.16 180)
